File: pcb/pcb.kicad_pcb (KiCad board)
At the start: 2 copper layers, 78 parts, among them J1 USB_C_Receptacle_USB2.0_16P, J2 F3311A7H121024E200, J3 Conn_01x02_Pin, J5 MSD-1-A, Q1 AO3400A, Q2 DMP3099L, Q3 DMP3099L, Q5 DMP3099L, SW1 SW_Push, SW2 SW_Push, SW3 SW_Push, SW4 SW_Push, SW5 SW_Push, SW6 SW_Push, SW7 SW_Push, SW8 SW_Push, SW9 SW_Push, U1 ESP32-C3-WROOM-02, U2 MCP73831-2-OT, U3 TCA9534, U4 AP2112K-3.3, U5 MAX17048G+T10, U6 USBLC6-2SC6, U7 TCA9534

Commit message: Place PCB components
Parts:
- removed R26: 10k, Resistor_SMD:R_0805_2012Metric_Pad1.20x1.40mm_HandSolder
- added R31: 10k, Resistor_SMD:R_0805_2012Metric_Pad1.20x1.40mm_HandSolder, F.Cu at (147.7, 57.4)
- moved Q1 179.9 mm to (93.3, 143.1)
- moved C5 167.6 mm to (93.1, 128.7)
- moved C6 167.4 mm to (93.1, 130.8)
- moved L1 167.3 mm to (96.3, 123.8)
- moved R5 163.3 mm to (93.1, 134.8)
- moved R6 162.0 mm to (93.0, 132.8)
- moved C8 157.7 mm to (99.1, 138.6)
- moved R7 154.1 mm to (99.0, 141.3)
- moved Q2 153.8 mm to (104.3, 140.4)
- moved D1 152.7 mm to (100.0, 128.0)
- moved D2 152.7 mm to (100.0, 131.3)
- moved D3 152.7 mm to (100.0, 134.7)
- moved U2 130.8 mm to (154.9, 100.5)
- moved J3 124.1 mm to (153.7, 107.4)
- moved J2 122.2 mm to (126.5, 141.6)
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Connections:
- net /V_BAT renamed +BATT
- net GND renamed -BATT
- SW5 pad 1: Net-(U3-P7) -> Net-(U7-P4)
- U3 pad 12: Net-(U3-P7) -> /SD_PWR
- U7 pad 9: /SD_PWR -> Net-(U7-P4)
Other:
- board outline added: 71.2 x 126.4 mm
- copper layers 2 -> 4
