File: pcb/pcb.kicad_sch (KiCad schematic)
At the start: 16 parts, among them J1 USB_C_Receptacle_USB2.0_16P, U1 ESP32-C3-WROOM-02, U2 AP2112K-3.3, U3 USBLC6-2SC6

Commit message: Assign footprints and organize pcb layout
Parts:
- removed U2: AP2112K-3.3, Package_TO_SOT_SMD:SOT-23-5, symbol Regulator_Linear:AP2112K-3.3
- removed U3: USBLC6-2SC6, Package_TO_SOT_SMD:SOT-23-6, symbol Power_Protection:USBLC6-2SC6
- added C10, C11, C16: 1uF/50V, Capacitor_SMD:C_0805_2012Metric_Pad1.18x1.45mm_HandSolder, symbol Device:C
- added C12, C13, C14, C15, C5, C6, C7: 4.7uF/25V, Capacitor_SMD:C_0805_2012Metric_Pad1.18x1.45mm_HandSolder, symbol Device:C
- added C17, C18: 4.7uF, Capacitor_SMD:C_0805_2012Metric_Pad1.18x1.45mm_HandSolder, symbol Device:C
- added C8: 100nF/50V, Capacitor_SMD:C_0805_2012Metric_Pad1.18x1.45mm_HandSolder, symbol Device:C
- added D1, D2, D3: MBR0530, Diode_SMD:D_SOD-123, symbol Diode:MBR0530
- added D4: D_Schottky, Diode_SMD:D_SOD-123, symbol Device:D_Schottky
- added J2: F3311A7H121024E200, F3311A7H121024E200:AMPHENOL_F3311A7H121024E200, symbol F3311A7H121024E200:F3311A7H121024E200
- added J3: Conn_01x02_Pin, Connector_JST:JST_PH_B2B-PH-K_1x02_P2.00mm_Vertical, symbol Connector:Conn_01x02_Pin
- added J5: MSD-1-A, MSD-1-A:CUI_MSD-1-A, symbol MSD-1-A:MSD-1-A
- added L1: 10uH, Inductor_SMD:L_Taiyo-Yuden_NR-24xx_HandSoldering, symbol Device:L
- added Q1: AO3400A, Package_TO_SOT_SMD:SOT-23, symbol Transistor_FET:AO3400A
- added Q2: DMP3099L, Package_TO_SOT_SMD:SOT-23, symbol Transistor_FET:Q_PMOS_GSD
- added Q3, Q5: DMP3099L, Package_TO_SOT_SMD:SOT-23, symbol Transistor_FET:DMP3099L
- added R10, R11: 22, Resistor_SMD:R_0805_2012Metric_Pad1.20x1.40mm_HandSolder, symbol Device:R
- added R13, R14, R15, R16, R18, R19, R20, R21, R22, R23, R24, R25, R26, R27, R28, R29, R30: 10k, Resistor_SMD:R_0805_2012Metric_Pad1.20x1.40mm_HandSolder, symbol Device:R
- added R5: 2.2, Resistor_SMD:R_0805_2012Metric_Pad1.20x1.40mm_HandSolder, symbol Device:R
- added R6: 1M, Resistor_SMD:R_0805_2012Metric_Pad1.20x1.40mm_HandSolder, symbol Device:R
- added R7: 47K, Resistor_SMD:R_0805_2012Metric_Pad1.20x1.40mm_HandSolder, symbol Device:R
- added R8: 2k, Resistor_SMD:R_0805_2012Metric_Pad1.20x1.40mm_HandSolder, symbol Device:R
- added R9: 100k, Resistor_SMD:R_0805_2012Metric_Pad1.20x1.40mm_HandSolder, symbol Device:R
- added SW1, SW2, SW3, SW4: SW_Push, Button_Switch_THT:SW_PUSH_6mm, symbol Switch:SW_Push
- added SW5, SW6, SW7, SW8, SW9: SW_Push, Button_Switch_THT:SW_Tactile_SPST_Angled_PTS645Vx39-2LFS, symbol Switch:SW_Push
- added U2: MCP73831-2-OT, Package_TO_SOT_SMD:SOT-23-5, symbol Battery_Management:MCP73831-2-OT
- added U3, U7: TCA9534, TCA9534DWR:SOIC127P1030X265-16N, symbol Interface_Expansion:TCA9534
- added U4: AP2112K-3.3, Package_TO_SOT_SMD:SOT-23-5, symbol Regulator_Linear:AP2112K-3.3
- added U5: MAX17048G+T10, MAX17048G_T10:21-0168E_T822-3_MXM-M, symbol 2026-07-17_22-13-49:MAX17048G+T10
- added U6: USBLC6-2SC6, Package_TO_SOT_SMD:SOT-23-6, symbol Power_Protection:USBLC6-2SC6
- C1, C2, C3: footprint (none) -> Capacitor_SMD:C_0805_2012Metric_Pad1.18x1.45mm_HandSolder
- C4: value 1uF -> 10pF; footprint (none) -> Capacitor_SMD:C_0805_2012Metric_Pad1.18x1.45mm_HandSolder
- J1: footprint (none) -> Connector_USB:USB_C_Receptacle_GCT_USB4105-xx-A_16P_TopMnt_Horizontal
- R1, R2, R3, R4: footprint (none) -> Resistor_SMD:R_0805_2012Metric_Pad1.20x1.40mm_HandSolder
- TP1, TP2, TP3, TP4: footprint (none) -> TestPoint:TestPoint_Pad_D1.5mm
Connections:
- net BOOT: now also C4.2, R4.2, TP3.1; no longer R4.1
- net GND: now also C10.1, C11.1, C12.1, C13.1, C14.1, C15.1, C16.1, C17.2, C18.1, C5.1, C7.1, C8.2, D3.1 (K), J2.17, J2.8, J3.1 (Pin_1), J5.6 (VSS), J5.G1 (COVER_GND), J5.G2 (COVER_GND__1), J5.G3 (COVER_GND__2), J5.G4 (COVER_GND__3), R5.2, R6.1, R8.2, R9.2, SW1.2, SW2.2, SW3.2, SW4.2, SW5.2, SW6.2, SW7.2, SW8.2, SW9.2, U2.2 (V_{SS}), U3.1 (A0), U3.2 (A1), U3.3 (A2), U3.8 (GND), U4.2 (GND), U5.1 (CTG), U5.4 (GND), U5.6 (QSTRT), U5.9 (EPAD), U6.2 (GND), U7.2 (A1), U7.3 (A2), U7.8 (GND)
- net USB_D+: now also R10.2
- net USB_D-: now also R11.2
- net EPD_CS: now reaches U1.10 (IO10)
- net EPD_CS: now also J2.12, R14.2
- net I2C_SDA: now reaches U1.15 (IO3)
- net I2C_SDA: now also R16.2, U3.15 (SDA), U5.8 (SDA), U7.15 (SDA)
- net SPI_MISO: now reaches U1.16 (IO2)
- net SPI_MISO: now also J5.7 (DAT0), R20.2
- net SD_CS: now reaches U1.17 (IO1)
- net SD_CS: now also J5.2 (CD/DAT3), R19.2
- net INT: now reaches U1.18 (IO0)
- net INT: now also R21.2, U3.13 (~{INT}), U7.13 (~{INT})
- net EN: now reaches C3.2, R3.2, TP1.1, U1.2 (EN)
- net I2C_SCL: now reaches U1.3 (IO4)
- net I2C_SCL: now also R13.2, U3.14 (SCL), U5.7 (SCL), U7.14 (SCL)
- net SPI_SCLK: now reaches U1.5 (IO6)
- net SPI_SCLK: now also J2.13, J5.5 (CLK)
- net SPI_MOSI: now reaches U1.6 (IO7)
- net SPI_MOSI: now also J2.14, J5.3 (CMD)
- net at U1.7 (IO8): now also R15.2
- net at J1.A6 (D+), J1.B6 (D+): now also U6.3 (I/O2)
- net at J1.A7 (D-), J1.B7 (D-): now also U6.1 (I/O1)
- net VBUS renamed +5V
- net +5V: now also C18.2, D4.2 (A), Q3.1 (G), R9.1, U2.4 (V_{DD}), U6.5 (VBUS); no longer C1.1
- net VCC_3v3 renamed +3V3
- net +3V3: now also R4.1, C8.1, Q2.2 (S), Q5.2 (S), R13.1, R14.1, R15.1, R16.1, R18.1, R19.1, R20.1, R21.1, R22.1, R23.1, R24.1, R25.1, R26.1, R27.1, R28.1, R29.1, R30.1, R7.2, U3.16 (VDD), U4.5 (VOUT), U7.1 (A0), U7.16 (VDD)
- new net: R10.1, U6.4 (I/O2)
- new net: R11.1, U6.6 (I/O1)
- new net: C6.1, D2.2 (A), D3.2 (A)
- new net: R28.2, SW7.1, U7.5 (P1)
- new net: R25.2, SW4.1, U3.11 (P6)
- new net: R30.2, SW9.1, U7.7 (P3)
- new net: R24.2, SW3.1, U3.10 (P5)
- new net: R22.2, SW1.1, U3.7 (P3)
- new net: C10.2, J2.18
- new net: C15.2, J2.20
- new net: C13.2, J2.22
- new net: C11.2, J2.24
- new net: C7.2, J2.5
- new net: R27.2, SW6.1, U7.4 (P0)
- new net: R8.1, U2.5 (PROG)
- new net: C6.2, D1.2 (A), L1.2, Q1.3 (D)
- new net: R26.2, SW5.1, U3.12 (P7)
- new net: R23.2, SW2.1, U3.9 (P4)
- new net: R29.2, SW8.1, U7.6 (P2)
- new net: C1.1, D4.1 (K), Q3.2 (S), U4.1 (VIN), U4.3 (EN)
- new net: J5.4 (VDD), Q5.3 (D)
- new net 3V3_OUT: C16.2, C5.2, J2.15, J2.16, L1.1, Q2.3 (D)
- new net EPD_BUSY: J2.9, U3.6 (P2)
- new net EPD_DC: J2.11, U3.4 (P0)
- new net EPD_RST: J2.10, U3.5 (P1)
- new net GDR: J2.2, Q1.1 (G), R6.2
- new net PWR: Q2.1 (G), R7.1
- new net RESE: J2.3, Q1.2 (S), R5.1
- new net SD_PWR: Q5.1 (G), R18.2, U7.9 (P4)
- new net VGH: C14.2, D1.1 (K), J2.21
- new net VGL: C12.2, D2.1 (K), J2.23
- new net V_BAT: C17.1, J3.2 (Pin_2), Q3.3 (D), U2.3 (V_{BAT}), U5.2 (CELL), U5.3 (VDD)
- no-connect marks 2 -> 18
Other:
- note added: "24 Pin Display FPC Connector Receptacle"
- note added: "Battery Monitor IC"
- note added: "Charging IC"
- note added: "Display Booster Circuit"
- note added: "Display Power Circuit"
- note added: "ESP-32 Microcontroller"
- note added: "IO Extenders"
- note added: "MicroSD Card Reader"
- note added: "NAV_BUTTONS"
- note added: "PG_TURN_BUTTONS"
- note added: "Power Path with 3V3 LDO Regulator"
- note added: "SLEEP_BUTTON"
- note added: "Strapping Pins/Troubleshooting"
- note added: "TSV Diode"
- note added: "USB-C"
- note added: "strapping pins (2, 8, 9)"
- moved on the sheet: C1, C2, C3, C4, J1, R1, R2, R3, R4, TP1, TP2, TP3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

Commit message: Place PCB components
Parts:
- removed R26: 10k, Resistor_SMD:R_0805_2012Metric_Pad1.20x1.40mm_HandSolder, symbol Device:R
- added R31: 10k, Resistor_SMD:R_0805_2012Metric_Pad1.20x1.40mm_HandSolder, symbol Device:R
Connections:
- net +3V3: now also R31.1
- net SD_PWR: now also U3.12 (P7); no longer U7.9 (P4)
- net at SW5.1: now also U7.9 (P4), R31.2; no longer U3.12 (P7)
- net GND renamed -BATT
- net V_BAT renamed +BATT
Other:
- moved on the sheet: SW5
